File: mydacboard.kicad_pcb (KiCad board)
At the start: 2 copper layers, 38.7 x 26.6 mm, 14 parts, among them J1 Conn_02x10_Odd_Even, U1 MAX9850, U2 myaudiojack

Commit message: Updated audiojack U->J ref
Parts:
- renumbered U2 to J2
